Commit message: add more arx robot

File: descriptions/ARXRobotics/r5_description/urdf/robot.urdf (robot description, URDF)
Before this commit: robot R5a, 11 links, 10 joints
Links:
- removed link base
- added link camera; collision mesh filename=../meshes/d405.obj; visual mesh filename=../meshes/d405.obj
- added link camera_support; collision mesh filename=../meshes/camera_support.obj; visual mesh filename=../meshes/camera_support.obj
- added link left_pad
- added link right_pad
- link base_link: geometry collision mesh filename=../meshes/base_link.obj; visual mesh filename=../meshes/base_link.obj
- link link1: geometry collision mesh filename=../meshes/link1.obj; visual mesh filename=../meshes/link1.obj
- link link2: geometry collision mesh filename=../meshes/link2.obj; visual mesh filename=../meshes/link2.obj
- link link3: geometry collision mesh filename=../meshes/link3.obj; visual mesh filename=../meshes/link3.obj
- link link4: geometry collision mesh filename=../meshes/link4.obj; visual mesh filename=../meshes/link4.obj
- link link5: geometry collision mesh filename=../meshes/link5.obj; visual mesh filename=../meshes/link5.obj
- link link6: geometry collision mesh filename=../meshes/link6.obj; visual mesh filename=../meshes/link6.obj
- link link7: geometry collision mesh filename=../meshes/link7.obj; visual mesh filename=../meshes/link7.obj
- link link8: geometry collision mesh filename=../meshes/link8.obj; visual mesh filename=../meshes/link8.obj
Joints:
- removed joint base_fixed
- added joint camera_fixed: type fixed, parent camera_support, child camera, origin xyz=0.0385 0 0.0475 rpy=0 0.523 0
- added joint camera_support_fixed: type fixed, parent link6, child camera_support, origin xyz=0.045 0 0.021
- added joint left_pad_joint: type fixed, parent link7, child left_pad, origin xyz=0.05843 -0.0249 0 rpy=0 0 0
- added joint right_pad_joint: type fixed, parent link8, child right_pad, origin xyz=0.05843 0.0249 0 rpy=0 0 0
- joint gripper_center_fixed: origin xyz=0.08657 0 0 rpy=0 0 0 -> xyz=0.145 0 0 rpy=0 0 0
- joint joint1: origin xyz=0 0 0.0565 rpy=0 0 0 -> xyz=0 0 0.0565
- joint joint2: origin xyz=0.02 0 0.047 rpy=0 0 0 -> xyz=0.02 0 0.047
- joint joint4: origin xyz=0.245 -5E-05 -0.06 rpy=0 0 0 -> xyz=0.245 -5E-05 -0.06
- joint joint5: origin xyz=0.0702 5E-05 -0.083391 rpy=0 0 0 -> xyz=0.0702 5E-05 -0.083391
- joint joint7: origin xyz=0 0.024896 -0.0002436 rpy=0 0 0 -> xyz=0.08657 0.024896 -0.0002436; parent gripper_center -> link6
- joint joint8: mimic (none) -> joint=joint7; origin xyz=0 -0.0249 -0.00024366 rpy=0 0 0 -> xyz=0.08657 -0.0249 -0.00024366; parent gripper_center -> link6

File: descriptions/ARXRobotics/r5_description/xacro/R5.xacro (robot description, xacro)
@@ -1,483 +1,470 @@
 <?xml version="1.0"?>
-<robot
-    name="R5a">
-  <material name="black">
-    <color rgba="0.1 0.1 0.1 1"/>
-  </material>
-  <material name="dark">
-    <color rgba="0.2 0.2 0.2 1"/>
-  </material>
-  <link name="base_link">
-    <inertial>
-      <origin
-          xyz="-0.00013359 6.672E-05 0.031672"
-          rpy="0 0 0"/>
-      <mass
-          value="0.42272"/>
-      <inertia
-          ixx="0.00019"
-          ixy="0.00000"
-          ixz="0.00000"
-          iyy="0.00019"
-          iyz="0.00000"
-          izz="0.00020"/>
-    </inertial>
-    <visual>
-      <origin
-          xyz="0 0 0"
-          rpy="0 0 0"/>
-      <geometry>
-        <mesh
-            filename="file://$(find r5_description)/meshes/base_link.STL"/>
-      </geometry>
-      <material name="black"/>
-    </visual>
-    <collision>
-      <origin
-          xyz="0 0 0"
-          rpy="0 0 0"/>
-      <geometry>
-        <mesh
-            filename="file://$(find r5_description)/meshes/base_link.STL"/>
-      </geometry>
-    </collision>
-  </link>
-  <link
-      name="link1">
-    <inertial>
-      <origin
-          xyz="0.0050395 -0.0077407 0.020897"
-          rpy="0 0 0"/>
-      <mass
-          value="0.096804"/>
-      <inertia
-          ixx="0.00011"
-          ixy="-0.00001"
-          ixz="0.00001"
-          iyy="0.00005"
-          iyz="-0.00001"
-          izz="0.00010"/>
-    </inertial>
-    <visual>
-      <origin
-          xyz="0 0 0"
-          rpy="0 0 0"/>
-      <geometry>
-        <mesh
-            filename="file://$(find r5_description)/meshes/link1.STL"/>
-      </geometry>
-      <material name="dark"/>
-    </visual>
-    <collision>
-      <origin
-          xyz="0 0 0"
-          rpy="0 0 0"/>
-      <geometry>
-        <mesh
-            filename="file://$(find r5_description)/meshes/link1.STL"/>
-      </geometry>
-    </collision>
-  </link>
-  <joint
-      name="joint1"
-      type="revolute">
-    <origin
-        xyz="0 0 0.0565"
-        rpy="0 0 0"/>
-    <parent
-        link="base_link"/>
-    <child
-        link="link1"/>
-    <axis
-        xyz="0 0 1"/>
-    <limit
-        lower="-2.618"
-        upper="2.168"
-        effort="100"
-        velocity="5"/>
-  </joint>
-  <link
-      name="link2">
-    <inertial>
-      <origin
-          xyz="-0.12992 -0.0011822 -2.6366E-05"
-          rpy="0 0 0"/>
-      <mass
-          value="1.1988"/>
-      <inertia
-          ixx="0.00065"
-          ixy="0.00008"
-          ixz="0.00000"
-          iyy="0.01647"
-          iyz="0.00000"
-          izz="0.01646"/>
-    </inertial>
-    <visual>
-      <origin
-          xyz="0 0 0"
-          rpy="0 0 0"/>
-      <geometry>
-        <mesh
-            filename="file://$(find r5_description)/meshes/link2.STL"/>
-      </geometry>
-      <material name="black"/>
-    </visual>
-    <collision>
-      <origin
-          xyz="0 0 0"
-          rpy="0 0 0"/>
-      <geometry>
-        <mesh
-            filename="file://$(find r5_description)/meshes/link2.STL"/>
-      </geometry>
-    </collision>
-  </link>
-  <joint
-      name="joint2"
-      type="revolute">
-    <origin
-        xyz="0.02 0 0.047"
-        rpy="0 0 0"/>
-    <parent
-        link="link1"/>
-    <child
-        link="link2"/>
-    <axis
-        xyz="0 1 0"/>
-    <limit
-        lower="0"
-        upper="3.66"
-        effort="100"
-        velocity="5"/>
-  </joint>
-  <link
-      name="link3">
-    <inertial>
-      <origin
-          xyz="0.16181 0.0011723 -0.05455"
-          rpy="0 0 0"/>
-      <mass
-          value="0.84082"/>
-      <inertia
-          ixx="0.00082"
-          ixy="0.00008"
-          ixz="-0.00074"
-          iyy="0.00849"
-          iyz="0.00001"
-          izz="0.00834"/>
-    </inertial>
-    <visual>
-      <origin
-          xyz="0 0 0"
-          rpy="0 0 0"/>
-      <geometry>
-        <mesh
-            filename="file://$(find r5_description)/meshes/link3.STL"/>
-      </geometry>
-      <material name="dark"/>
-    </visual>
-    <collision>
-      <origin
-          xyz="0 0 0"
-          rpy="0 0 0"/>
-      <geometry>
-        <mesh
-            filename="file://$(find r5_description)/meshes/link3.STL"/>
-      </geometry>
-    </collision>
-  </link>
-  <joint
-      name="joint3"
-      type="revolute">
-    <origin
-        xyz="-0.264 0 0"
-        rpy="-3.1416 0 0"/>
-    <parent
-        link="link2"/>
-    <child
-        link="link3"/>
-    <axis
-        xyz="0 1 0"/>
-    <limit
-        lower="0"
-        upper="3.14"
-        effort="100"
-        velocity="5"/>
-  </joint>
-  <link
-      name="link4">
-    <inertial>
-      <origin
-          xyz="0.041751 0.0054236 -0.03337"
-          rpy="0 0 0"/>
-      <mass
-          value="0.12432"/>
-      <inertia
-          ixx="0.00022"
-          ixy="-0.00002"
-          ixz="-0.00009"
-          iyy="0.00025"
-          iyz="0.00002"
-          izz="0.00017"/>
-    </inertial>
-    <visual>
-      <origin
-          xyz="0 0 0"
-          rpy="0 0 0"/>
-      <geometry>
-        <mesh
-            filename="file://$(find r5_description)/meshes/link4.STL"/>
-      </geometry>
-      <material name="black"/>
-    </visual>
-    <collision>
-      <origin
-          xyz="0 0 0"
-          rpy="0 0 0"/>
-      <geometry>
-        <mesh
-            filename="file://$(find r5_description)/meshes/link4.STL"/>
-      </geometry>
-    </collision>
-  </link>
-  <joint
-      name="joint4"
-      type="revolute">
-    <origin
-        xyz="0.245 -5E-05 -0.06"
-        rpy="0 0 0"/>
-    <parent
-        link="link3"/>
-    <child
-        link="link4"/>
-    <axis
-        xyz="0 1 0"/>
-    <limit
-        lower="-1.57"
-        upper="1.57"
-        effort="100"
-        velocity="5"/>
-  </joint>
-  <link
-      name="link5">
-    <inertial>
-      <origin
-          xyz="-8.3435E-05 -1.5428E-05 0.052216"
-          rpy="0 0 0"/>
-      <mass
-          value="0.63601"/>
-      <inertia
-          ixx="0.00084"
-          ixy="0.00000"
-          ixz="0.00007"
-          iyy="0.00082"
-          iyz="0.00000"
-          izz="0.00026"/>
-    </inertial>
-    <visual>
-      <origin
-          xyz="0.0037 0 0"
-          rpy="0 0 0"/>
-      <geometry>
-        <mesh
-            filename="file://$(find r5_description)/meshes/link5.STL"/>
-      </geometry>
-      <material name="dark"/>
-    </visual>
-    <collision>
-      <origin
-          xyz="0 0 0"
-          rpy="0 0 0"/>
-      <geometry>
-        <mesh
-            filename="file://$(find r5_description)/meshes/link5.STL"/>
-      </geometry>
-    </collision>
-  </link>
-  <joint
-      name="joint5"
-      type="revolute">
-    <origin
-        xyz="0.0702 5E-05 -0.083391"
-        rpy="0 0 0"/>
-    <parent
-        link="link4"/>
-    <child
-        link="link5"/>
-    <axis
-        xyz="0 0 1"/>
-    <limit
-        lower="-1.57"
-        upper="1.57"
-        effort="100"
-        velocity="5"/>
-  </joint>
-  <link
-      name="link6">
-    <inertial>
-      <origin
-          xyz="0.041697 2.4368E-05 0.00014464"
-          rpy="0 0 0"/>
-      <mass
-          value="0.44089"/>
-      <inertia
-          ixx="0.00038"
-          ixy="0.00000"
-          ixz="0.00000"
-          iyy="0.00028"
-          iyz="0.00000"
-          izz="0.00050"/>
-    </inertial>
-    <visual>
-      <origin
-          xyz="0 0 0"
-          rpy="0 0 0"/>
-      <geometry>
-        <mesh
-            filename="file://$(find r5_description)/meshes/link6.STL"/>
-      </geometry>
-      <material name="black"/>
-    </visual>
-    <collision>
-      <origin
-          xyz="0 0 0"
-          rpy="0 0 0"/>
-      <geometry>
-        <mesh
-            filename="file://$(find r5_description)/meshes/link6.STL"/>
-      </geometry>
-    </collision>
-  </link>
-  <joint
-      name="joint6"
-      type="revolute">
-    <origin
-        xyz="0.025286 0 0.083391"
-        rpy="3.1416 0 0"/>
-    <parent
-        link="link5"/>
-    <child
-        link="link6"/>
-    <axis
-        xyz="1 0 0"/>
-    <limit
-        lower="-1.57"
-        upper="1.57"
-        effort="100"
-        velocity="5"/>
-  </joint>
-  <link
-      name="link7">
-    <inertial>
-      <origin
-          xyz="-0.00035522 -0.007827 -0.0029883"
-          rpy="0 0 0"/>
-      <mass
-          value="0.064798"/>
-      <inertia
-          ixx="0.00002"
-          ixy="0.00000"
-          ixz="0.00000"
-          iyy="0.00003"
-          iyz="0.00000"
-          izz="0.00003"/>
-    </inertial>
-    <visual>
-      <origin
-          xyz="0 0 0"
-          rpy="0 0 0"/>
-      <geometry>
-        <mesh
-            filename="file://$(find r5_description)/meshes/link7.STL"/>
-      </geometry>
-      <material name="dark"/>
-    </visual>
-    <collision>
-      <origin
-          xyz="0 0 0"
-          rpy="0 0 0"/>
-      <geometry>
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