Commit message: add aloha2 and piper

File: descriptions/ARXRobotics/r5_description/xacro/R5.xacro (robot description, xacro)
@@ -467,4 +467,41 @@
       <origin xyz="0.08657 0 0" rpy="0 0 0"/>
     </joint>
+    <link name="${prefix}left_pad"/>
+    <joint name="${prefix}left_pad_joint" type="fixed">
+      <parent link="${prefix}link7"/>
+      <child link="${prefix}left_pad"/>
+      <origin xyz="0.05843 -0.0249 0" rpy="0 0 0"/>
+    </joint>
+    <link name="${prefix}right_pad"/>
+    <joint name="${prefix}right_pad_joint" type="fixed">
+      <parent link="${prefix}link8"/>
+      <child link="${prefix}right_pad"/>
+      <origin xyz="0.05843 0.0249 0" rpy="0 0 0"/>
+    </joint>
+    <link name="${prefix}camera_support">
+      <visual>
+        <geometry>
+          <mesh filename="file://$(find x5_description)/meshes/camera_support.obj"/>
+        </geometry>
+      </visual>
+    </link>
+    <joint name="${prefix}camera_support_fixed" type="fixed">
+      <parent link="${prefix}link6"/>
+      <child link="${prefix}camera_support"/>
+      <origin xyz="0.045 0 0.021"/>
+    </joint>
+    <link name="${prefix}camera">
+      <visual>
+        <geometry>
+          <mesh
+              filename="file://$(find x5_description)/meshes/d405.obj"/>
+        </geometry>
+      </visual>
+    </link>
+    <joint name="${prefix}camera_fixed" type="fixed">
+      <origin xyz="0.0385 0 0.0475" rpy="0 0.523 0"/>
+      <parent link="${prefix}camera_support"/>
+      <child link="${prefix}camera"/>
+    </joint>
   </xacro:macro>
 </robot>

File: descriptions/ARXRobotics/x5_description/xacro/X5.xacro (robot description, xacro)
@@ -481,10 +481,6 @@
     <link name="${prefix}camera_support">
       <visual>
-        <origin
-            xyz="0 0 0"
-            rpy="0 0 0"/>
-        <geometry>
-          <mesh
-              filename="file://$(find x5_description)/meshes/camera_support.obj"/>
+        <geometry>
+          <mesh filename="file://$(find x5_description)/meshes/camera_support.obj"/>
         </geometry>
       </visual>
@@ -504,10 +500,7 @@
     </link>
     <joint name="${prefix}camera_fixed" type="fixed">
-      <origin
-          xyz="0.0385 0 0.0475"
-          rpy="0 0.523 0"/>
+      <origin xyz="0.0385 0 0.0475" rpy="0 0.523 0"/>
       <parent link="${prefix}camera_support"/>
       <child link="${prefix}camera"/>
-      <origin xyz="0.045 0 0.021"/>
     </joint>
   </xacro:macro>
