Commit message: ocs controller init

File: moveit/Dobot/cr5_moveit_config/xacro/robot.xacro (robot description, xacro)
@@ -1,34 +1,5 @@
 <?xml version="1.0"?>
 <robot xmlns:xacro="http://www.ros.org/wiki/xacro" name="CR5">
-  <xacro:arg name="ros2_control_hardware_type" default="mock_components"/>
-  <link name="world"/>
-  <joint name="world_fixed" type="fixed">
-    <parent link="world"/>
-    <child link="base_link"/>
-    <origin xyz="0.0 0.0 0.0" rpy="0 0 0"/>
-  </joint>
-  <xacro:include filename="$(find cr5_description)/xacro/arm.xacro"/>
-  <xacro:CR5 name=""/>
   <!-- Import R5 ros2_control description -->
-  <xacro:include filename="$(find cr5_description)/xacro/ros2_control/cr5.ros2_control.xacro"/>
-  <xacro:cr5_system name="cr5System" ros2_control_hardware_type="$(arg ros2_control_hardware_type)"/>
-  <xacro:arg name="type" default="robotiq85"/>
-  <xacro:if value="${'$(arg type)' == 'robotiq85'}">
-    <joint name="gripper_fix" type="fixed">
-      <parent link="Link6"/>
-      <child link="eef_base_link"/>
-    </joint>
-    <xacro:include filename="$(find robotiq_description)/xacro/robotiq85.xacro"/>
-    <xacro:Robotiq85 name="eef"/>
-    <xacro:include filename="$(find robotiq_description)/xacro/ros2_control/robotiq85.ros2_control.xacro"/>
-    <xacro:robotiq85_system name="robotiq85System" ros2_control_hardware_type="$(arg ros2_control_hardware_type)"/>
-  </xacro:if>
-  <xacro:arg name="gazebo" default="false"/>
-  <xacro:if value="$(arg gazebo)">
-    <gazebo>
-      <plugin filename="gz_ros2_control-system" name="gz_ros2_control::GazeboSimROS2ControlPlugin">
-        <parameters>$(find cr5_moveit_config)/config/ros2_controllers.yaml</parameters>
-      </plugin>
-    </gazebo>
-  </xacro:if>
+  <xacro:include filename="$(find cr5_description)/xacro/ros2_control/robot.xacro"/>
 </robot>
